Commit message: Integrated grippers kg2 and R85 to 7DoF model

File: movo_common/movo_description/urdf/manipulation/kinova_grippers/kg2_gripper.urdf.xacro (robot description, xacro)
@@ -37,5 +37,5 @@
             <minDepth>0.0001</minDepth>
         </gazebo>
-        <joint name="${prefix}gripper_finger2_joint" type="prismatic">
+        <joint name="${prefix}gripper_finger2_joint" type="revolute">
             <parent link="${prefix}gripper_base_link"/>
             <child link="${prefix}gripper_finger2_knuckle_link"/>
@@ -73,5 +73,5 @@
             <minDepth>0.0001</minDepth>
         </gazebo>
-        <joint name="${prefix}gripper_finger1_joint" type="prismatic">
+        <joint name="${prefix}gripper_finger1_joint" type="revolute">
             <parent link="${prefix}gripper_base_link"/>
             <child link="${prefix}gripper_finger1_knuckle_link"/>
