Commit message: **Work in progress** Pick and Place demo in 7DoF works with both Gazebo and the real MOVO

File: movo_common/movo_description/urdf/manipulation/jaco/jaco_7dof.urdf.xacro (robot description, xacro)
@@ -43,7 +43,16 @@
     <property name="arm_half_joint_rpy" value="-${M_PI/2} 0 0" />
     <property name="elbow_joint_rpy" value="-${M_PI/2} 0 0"/>
+    <property name="wrist_spherical_1_joint_rpy" value="${M_PI/2} ${M_PI} 0" />
+    <property name="wrist_spherical_2_joint_rpy" value="-${M_PI/2} 0 0" />
+    <property name="wrist_3_joint_rpy" value="${M_PI/2} 0 0" />
+    <!--
+    <property name="shoulder_pan_joint_rpy" value="0 ${M_PI} 0" />
+    <property name="shoulder_lift_joint_rpy" value="${M_PI/2} 0 0" />
+    <property name="arm_half_joint_rpy" value="-${M_PI/2} ${M_PI} 0" />
+    <property name="elbow_joint_rpy" value="-${M_PI/2} 0 0"/>
     <property name="wrist_spherical_1_joint_rpy" value="${M_PI/2} 0 0" />
     <property name="wrist_spherical_2_joint_rpy" value="-${M_PI/2} 0 0" />
-    <property name="wrist_3_joint_rpy" value="${M_PI/2} 0 0" />
+    <property name="wrist_3_joint_rpy" value="${M_PI/2} ${M_PI} 0" />
+     -->
     <xacro:macro name="jaco_robot_7dof" params="prefix parent *origin">
         <joint name="${prefix}kinova_joint" type="fixed">
@@ -55,10 +64,10 @@
             <visual>
                 <geometry>
-                <mesh filename="package://movo_description/meshes/manipulation/jaco/visual/base.dae"/>
-                </geometry>
-            </visual>
-            <collision>
-                <geometry>
-                <mesh filename="package://movo_description/meshes/manipulation/jaco/collision/base.stl"/>
+                <mesh filename="package://movo_description/meshes/manipulation/jaco/visual/base_7dof.dae"/>
+                </geometry>
+            </visual>
+            <collision>
+                <geometry>
+                <mesh filename="package://movo_description/meshes/manipulation/jaco/collision/base_7dof.stl"/>
                 </geometry>
             </collision>
@@ -91,10 +100,10 @@
             <visual>
                 <geometry>
-                    <mesh filename="package://movo_description/meshes/manipulation/jaco/visual/shoulder.dae"/>
-                </geometry>
-            </visual>
-            <collision>
-                <geometry>
-                    <mesh filename="package://movo_description/meshes/manipulation/jaco/collision/shoulder.stl"/>
+                    <mesh filename="package://movo_description/meshes/manipulation/jaco/visual/shoulder_7dof.dae"/>
+                </geometry>
+            </visual>
+            <collision>
+                <geometry>
+                    <mesh filename="package://movo_description/meshes/manipulation/jaco/collision/shoulder_7dof.stl"/>
                 </geometry>
             </collision>
@@ -132,5 +141,5 @@
             <collision>
                 <geometry>
-                    <mesh filename="package://movo_description/meshes/manipulation/jaco/visual/arm_half_1.dae"/>
+                    <mesh filename="package://movo_description/meshes/manipulation/jaco/collision/arm_half_1.stl"/>
                 </geometry>
             </collision>
@@ -157,5 +166,5 @@
             <origin xyz="0 -0.205 0" rpy="${arm_half_joint_rpy}"/>
             <axis xyz="0 0 1" />
-            <limit lower="-2.238" upper="2.238" effort="30000.5" velocity="0.691150384"/>
+            <limit lower="${-M_PI}" upper="${M_PI}" effort="30000.5" velocity="0.691150384"/>
             <dynamics damping="0.01" friction="0.0"/>
         </joint>
@@ -168,5 +177,5 @@
             <collision>
                 <geometry>
-                    <mesh filename="package://movo_description/meshes/manipulation/jaco/visual/arm_half_2.dae"/>
+                    <mesh filename="package://movo_description/meshes/manipulation/jaco/collision/arm_half_2.stl"/>
                 </geometry>
             </collision>
@@ -199,10 +208,10 @@
             <visual>
                 <geometry>
-                    <mesh filename="package://movo_description/meshes/manipulation/jaco/visual/forearm.dae"/>
-                </geometry>
-            </visual>
-            <collision>
-                <geometry>
-                    <mesh filename="package://movo_description/meshes/manipulation/jaco/collision/forearm.stl"/>
+                    <mesh filename="package://movo_description/meshes/manipulation/jaco/visual/forearm_7dof.dae"/>
+                </geometry>
+            </visual>
+            <collision>
+                <geometry>
+                    <mesh filename="package://movo_description/meshes/manipulation/jaco/collision/forearm_7dof.stl"/>
                 </geometry>
             </collision>
@@ -218,5 +227,6 @@
             <parent link="${prefix}forearm_link" />
             <child link="${prefix}wrist_spherical_1_link" />
-            <origin xyz="0 0.20725 0 " rpy="${wrist_spherical_1_joint_rpy}" />
+          <!--  <origin xyz="0 0.20725 0 " rpy="${wrist_spherical_1_joint_rpy}" /> -->
+            <origin xyz="0 0.2073 -0.0114" rpy="${wrist_spherical_1_joint_rpy}" />
             <axis xyz="0 0 1" />
             <limit lower="${-M_PI}" upper="${M_PI}" effort="60000.8" velocity="0.921533845"/>
@@ -231,5 +241,5 @@
             <collision>
                 <geometry>
-                    <mesh filename="package://movo_description/meshes/manipulation/jaco/visual/wrist_spherical_1.dae"/>
+                    <mesh filename="package://movo_description/meshes/manipulation/jaco/collision/wrist_spherical_1.stl"/>
                 </geometry>
             </collision>
@@ -256,5 +266,5 @@
             <origin xyz="0 0 -0.10375 " rpy="${wrist_spherical_2_joint_rpy}" />
             <axis xyz="0 0 1" />
-            <limit lower="${-M_PI}" upper="${M_PI}" effort="60000.8" velocity="0.921533845"/>
+            <limit lower="${-2.78}" upper="${2.78}" effort="60000.8" velocity="0.921533845"/>
             <dynamics damping="0.01" friction="0.0"/>
         </joint>
@@ -267,5 +277,5 @@
             <collision>
                 <geometry>
-                    <mesh filename="package://movo_description/meshes/manipulation/jaco/visual/wrist_spherical_2.dae"/>
+                    <mesh filename="package://movo_description/meshes/manipulation/jaco/collision/wrist_spherical_2.stl"/>
                 </geometry>
             </collision>
@@ -308,5 +318,5 @@
             <inertial>
                 <mass value="${wrist_3_mass}" />
-                <origin xyz="0 0 -0.06" />
+                <origin xyz="-0.00082 0.000048 -0.216121" />
                 <inertia  ixx="0.000048"  ixy="0.000000"  ixz="0.000000"
                           iyx="0.000000"  iyy="0.000049"  iyz="0.000000"
@@ -327,7 +337,4 @@
             <child link="${prefix}ee_link" />
             <origin xyz="0 0 -0.1600" rpy="${M_PI} ${M_PI/2} 0"/>
-            <!--
-            <origin xyz="0 0 -0.202757" rpy="${M_PI} ${M_PI/2} 0"/>
-            -->
         </joint>
         <link name="${prefix}ee_link"/>

File: movo_common/movo_description/urdf/manipulation/kinova_grippers/kg2_gripper.urdf.xacro (robot description, xacro)
@@ -37,5 +37,5 @@
             <minDepth>0.0001</minDepth>
         </gazebo>
-        <joint name="${prefix}gripper_finger2_joint" type="revolute">
+        <joint name="${prefix}gripper_finger2_joint" type="prismatic">
             <parent link="${prefix}gripper_base_link"/>
             <child link="${prefix}gripper_finger2_knuckle_link"/>
@@ -73,5 +73,5 @@
             <minDepth>0.0001</minDepth>
         </gazebo>
-        <joint name="${prefix}gripper_finger1_joint" type="revolute">
+        <joint name="${prefix}gripper_finger1_joint" type="prismatic">
             <parent link="${prefix}gripper_base_link"/>
             <child link="${prefix}gripper_finger1_knuckle_link"/>

File: movo_common/movo_description/urdf/movo.urdf.xacro (robot description, xacro)
@@ -32,8 +32,4 @@
     <xacro:include filename="$(find movo_description)/urdf/movo_components/movo_pan_tilt.urdf.xacro" />
     <xacro:include filename="$(find movo_description)/urdf/movo_components/movo_body.urdf.xacro" />
-    <!--
-    <xacro:include filename="$(find movo_description)/urdf/manipulation/jaco/jaco.urdf.xacro" />
-    <xacro:include filename="$(find movo_description)/urdf/manipulation/jaco/jaco_7dof.urdf.xacro" />
-    -->
     <xacro:include filename="$(find movo_description)/urdf/manipulation/robotiq/robotiq_85_gripper.urdf.xacro" />
     <xacro:include filename="$(find movo_description)/urdf/manipulation/kinova_grippers/kg3_gripper.urdf.xacro" />
@@ -76,8 +72,8 @@
     	<xacro:if value="$(optenv MOVO_HAS_KINOVA_ARM_7DOF false)">
     		<xacro:include filename="$(find movo_description)/urdf/manipulation/jaco/jaco_7dof.urdf.xacro" />
+            <xacro:jaco_robot_7dof prefix="right_" parent="linear_actuator_link">
+            <origin xyz="0.0261046 -0.13335 0.2799937" rpy="${-M_PI/2} 0 ${-M_PI/2}"/>
+            </xacro:jaco_robot_7dof>
             <xacro:jaco_robot_7dof prefix="left_" parent="linear_actuator_link">
-                <origin xyz="0.0261046 -0.13335 0.2799937" rpy="${-M_PI/2} 0 ${-M_PI/2}"/>
-            </xacro:jaco_robot_7dof>
-            <xacro:jaco_robot_7dof prefix="right_" parent="linear_actuator_link">
                 <origin xyz="0.0261046 0.13335 0.2799937" rpy="${-M_PI/2} 0 ${-M_PI/2}"/>
             </xacro:jaco_robot_7dof>

Commit message: Cleanup

File: movo_common/movo_description/urdf/manipulation/jaco/jaco_7dof.urdf.xacro (robot description, xacro)
@@ -46,13 +46,4 @@
     <property name="wrist_spherical_2_joint_rpy" value="-${M_PI/2} 0 0" />
     <property name="wrist_3_joint_rpy" value="${M_PI/2} ${M_PI} 0" />
-    <!--
-    <property name="shoulder_pan_joint_rpy" value="0 ${M_PI} 0" />
-    <property name="shoulder_lift_joint_rpy" value="${M_PI/2} 0 0" />
-    <property name="arm_half_joint_rpy" value="-${M_PI/2} ${M_PI} 0" />
-    <property name="elbow_joint_rpy" value="-${M_PI/2} 0 0"/>
-    <property name="wrist_spherical_1_joint_rpy" value="${M_PI/2} 0 0" />
-    <property name="wrist_spherical_2_joint_rpy" value="-${M_PI/2} 0 0" />
-    <property name="wrist_3_joint_rpy" value="${M_PI/2} ${M_PI} 0" />
-     -->
     <xacro:macro name="jaco_robot_7dof" params="prefix parent *origin">
         <joint name="${prefix}kinova_joint" type="fixed">
@@ -64,10 +55,10 @@
             <visual>
                 <geometry>
-                <mesh filename="package://movo_description/meshes/manipulation/jaco/visual/base_7dof.dae"/>
-                </geometry>
-            </visual>
-            <collision>
-                <geometry>
-                <mesh filename="package://movo_description/meshes/manipulation/jaco/collision/base_7dof.stl"/>
+                <mesh filename="package://movo_description/meshes/manipulation/jaco/visual/base.dae"/>
+                </geometry>
+            </visual>
+            <collision>
+                <geometry>
+                <mesh filename="package://movo_description/meshes/manipulation/jaco/collision/base.stl"/>
                 </geometry>
             </collision>
