Commit message: modified files first implementation untested

File: movo_common/movo_description/urdf/gzplugin_grasp_fix.urdf.xacro (robot description, xacro)
@@ -28,6 +28,10 @@
 -->
 <robot name="movo_gripper_fix" xmlns:xacro="http://ros.org/wiki/xacro">
+    <xacro:property name="right_6dof_arm" value="$(optenv MOVO_HAS_RIGHT_ARM_6DOF false)"/>
+    <xacro:property name="right_7dof_arm" value="$(optenv MOVO_HAS_RIGHT_ARM_7DOF false)"/>
+    <xacro:property name="left_6dof_arm" value="$(optenv MOVO_HAS_LEFT_ARM_6DOF false)"/>
+    <xacro:property name="left_7dof_arm" value="$(optenv MOVO_HAS_LEFT_ARM_7DOF false)"/>
     <xacro:macro name="gzplugin_grasp_fix">
-        <xacro:if value="$(optenv MOVO_HAS_KINOVA_ARM false)">
+        <xacro:if value="${(right_6dof_arm=='true') or (right_7dof_arm=='true')}">
             <xacro:if value="$(optenv MOVO_HAS_RIGHT_ROBOTIQ_GRIPPER false)">
                 <gazebo>
@@ -55,5 +59,65 @@
                 </gazebo>
             </xacro:if>
-            <xacro:if value="$(optenv MOVO_HAS_LEFT_ROBOTIQ_GRIPPER false)">
+            <xacro:if value="$(optenv MOVO_HAS_RIGHT_KG2_GRIPPER false)">
+                <gazebo>
+                    <plugin name="gazebo_right_grasp_fix" filename="libgazebo_grasp_fix.so">
+                        <arm>
+                            <arm_name>right_arm</arm_name>
+                            <palm_link>right_wrist_3_link</palm_link>
+                            <gripper_link>right_gripper_finger1_knuckle_link</gripper_link>
+                            <gripper_link>right_gripper_finger2_knuckle_link</gripper_link>
+                        </arm>
+                        <forces_angle_tolerance>100</forces_angle_tolerance>
+                        <update_rate>50</update_rate>
+                        <grip_count_threshold>1</grip_count_threshold>
+                        <max_grip_count>2</max_grip_count>
+                        <release_tolerance>0.006</release_tolerance>
+                        <disable_collisions_on_attach>true</disable_collisions_on_attach>
+                        <contact_topic>right_gripper/contacts</contact_topic>
+                    </plugin>
+                </gazebo>
+            </xacro:if>
+            <xacro:if value="$(optenv MOVO_HAS_RIGHT_KG3_GRIPPER false)">
+                <gazebo>
+                    <plugin name="gazebo_right_grasp_fix" filename="libgazebo_grasp_fix.so">
+                        <arm>
+                            <arm_name>right_arm</arm_name>
+                            <palm_link> right_wrist_3_link </palm_link>
+                            <gripper_link> right_gripper_finger1_knuckle_link </gripper_link>
+                            <gripper_link> right_gripper_finger2_knuckle_link </gripper_link>
+                            <gripper_link> right_gripper_finger3_knuckle_link </gripper_link>
+                        </arm>
+                        <forces_angle_tolerance>100</forces_angle_tolerance>
+                        <update_rate>50</update_rate>
+                        <grip_count_threshold>1</grip_count_threshold>
+                        <max_grip_count>8</max_grip_count>
+                        <release_tolerance>0.006</release_tolerance>
+                        <disable_collisions_on_attach>true</disable_collisions_on_attach>
+                        <contact_topic>right_gripper/contacts</contact_topic>
+                    </plugin>
+                </gazebo>
+            </xacro:if>
+        </xacro:if>
+        <xacro:if value="${(left_6dof_arm=='true') or (left_7dof_arm=='true')}">
+            <xacro:if value="$(optenv MOVO_HAS_LEFT_KG2_GRIPPER false)">
+                <gazebo>
+                    <plugin name="gazebo_left_grasp_fix" filename="libgazebo_grasp_fix.so">
+                        <arm>
+                            <arm_name>left_arm</arm_name>
+                            <palm_link>left_wrist_3_link</palm_link>
+                            <gripper_link>left_gripper_finger1_knuckle_link</gripper_link>
+                            <gripper_link>left_gripper_finger2_knuckle_link</gripper_link>
+                        </arm>
+                        <forces_angle_tolerance>100</forces_angle_tolerance>
+                        <update_rate>50</update_rate>
+                        <grip_count_threshold>1</grip_count_threshold>
+                        <max_grip_count>2</max_grip_count>
+                        <release_tolerance>0.006</release_tolerance>
+                        <disable_collisions_on_attach>true</disable_collisions_on_attach>
+                        <contact_topic>left_gripper/contacts</contact_topic>
+                    </plugin>
+                </gazebo>
+            </xacro:if>
+	    <xacro:if value="$(optenv MOVO_HAS_LEFT_ROBOTIQ_GRIPPER false)">
                 <gazebo>
                     <plugin name="gazebo_left_grasp_fix" filename="libgazebo_grasp_fix.so">
@@ -77,62 +141,4 @@
                         <disable_collisions_on_attach>true</disable_collisions_on_attach>
                         <contact_topic>left_gripper/contacts</contact_topic>
-                    </plugin>
-                </gazebo>
-            </xacro:if>
-            <xacro:if value="$(optenv MOVO_HAS_RIGHT_KG2_GRIPPER false)">
-                <gazebo>
-                    <plugin name="gazebo_right_grasp_fix" filename="libgazebo_grasp_fix.so">
-                        <arm>
-                            <arm_name>right_arm</arm_name>
-                            <palm_link>right_wrist_3_link</palm_link>
-                            <gripper_link>right_gripper_finger1_knuckle_link</gripper_link>
-                            <gripper_link>right_gripper_finger2_knuckle_link</gripper_link>
-                        </arm>
-                        <forces_angle_tolerance>100</forces_angle_tolerance>
-                        <update_rate>50</update_rate>
-                        <grip_count_threshold>1</grip_count_threshold>
-                        <max_grip_count>2</max_grip_count>
-                        <release_tolerance>0.006</release_tolerance>
-                        <disable_collisions_on_attach>true</disable_collisions_on_attach>
-                        <contact_topic>right_gripper/contacts</contact_topic>
-                    </plugin>
-                </gazebo>
-            </xacro:if>
-            <xacro:if value="$(optenv MOVO_HAS_LEFT_KG2_GRIPPER false)">
-                <gazebo>
-                    <plugin name="gazebo_left_grasp_fix" filename="libgazebo_grasp_fix.so">
-                        <arm>
-                            <arm_name>left_arm</arm_name>
-                            <palm_link>left_wrist_3_link</palm_link>
-                            <gripper_link>left_gripper_finger1_knuckle_link</gripper_link>
-                            <gripper_link>left_gripper_finger2_knuckle_link</gripper_link>
-                        </arm>
-                        <forces_angle_tolerance>100</forces_angle_tolerance>
-                        <update_rate>50</update_rate>
-                        <grip_count_threshold>1</grip_count_threshold>
-                        <max_grip_count>2</max_grip_count>
-                        <release_tolerance>0.006</release_tolerance>
-                        <disable_collisions_on_attach>true</disable_collisions_on_attach>
-                        <contact_topic>left_gripper/contacts</contact_topic>
-                    </plugin>
-                </gazebo>
-            </xacro:if>
-            <xacro:if value="$(optenv MOVO_HAS_RIGHT_KG3_GRIPPER false)">
-                <gazebo>
-                    <plugin name="gazebo_right_grasp_fix" filename="libgazebo_grasp_fix.so">
-                        <arm>
-                            <arm_name>right_arm</arm_name>
-                            <palm_link> right_wrist_3_link </palm_link>
-                            <gripper_link> right_gripper_finger1_knuckle_link </gripper_link>
-                            <gripper_link> right_gripper_finger2_knuckle_link </gripper_link>
-                            <gripper_link> right_gripper_finger3_knuckle_link </gripper_link>
-                        </arm>
-                        <forces_angle_tolerance>100</forces_angle_tolerance>
-                        <update_rate>50</update_rate>
-                        <grip_count_threshold>1</grip_count_threshold>
-                        <max_grip_count>8</max_grip_count>
-                        <release_tolerance>0.006</release_tolerance>
-                        <disable_collisions_on_attach>true</disable_collisions_on_attach>
-                        <contact_topic>right_gripper/contacts</contact_topic>
                     </plugin>
                 </gazebo>

File: movo_common/movo_description/urdf/movo.urdf.xacro (robot description, xacro)
@@ -69,25 +69,42 @@
     </xacro:if>
     <!-- Arms -->
-    <xacro:if value="$(optenv MOVO_HAS_KINOVA_ARM false)">
-    	<xacro:if value="$(optenv MOVO_HAS_KINOVA_ARM_7DOF false)">
-    		<xacro:include filename="$(find movo_description)/urdf/manipulation/jaco/jaco_7dof.urdf.xacro" />
-            <xacro:jaco_robot_7dof prefix="right_" parent="linear_actuator_link">
-            <origin xyz="0.0261046 -0.13335 0.2799937" rpy="${-M_PI/2} 0 ${-M_PI/2}"/>
-            </xacro:jaco_robot_7dof>
-            <xacro:jaco_robot_7dof prefix="left_" parent="linear_actuator_link">
-                <origin xyz="0.0261046 0.13335 0.2799937" rpy="${-M_PI/2} 0 ${-M_PI/2}"/>
-            </xacro:jaco_robot_7dof>
-        </xacro:if>
-        <xacro:if value="$(optenv MOVO_HAS_KINOVA_ARM_6DOF false)">
-        	<xacro:include filename="$(find movo_description)/urdf/manipulation/jaco/jaco.urdf.xacro" />
-            <xacro:jaco_robot prefix="right_" parent="linear_actuator_link">
-		        <origin xyz="0.0261046 -0.13335 0.2799937" rpy="${-M_PI/2} 0 ${-M_PI/2}"/>
+	<xacro:if value="$(optenv MOVO_HAS_RIGHT_ARM_7DOF false)">  <!-- movo has a right arm of 7 dof type -->
+		<xacro:include filename="$(find movo_description)/urdf/manipulation/jaco/jaco_7dof.urdf.xacro" />
+		<xacro:jaco_robot_7dof prefix="right_" parent="linear_actuator_link">
+		   <origin xyz="0.0261046 -0.13335 0.2799937" rpy="${-M_PI/2} 0 ${-M_PI/2}"/>
+		</xacro:jaco_robot_7dof>
+		<xacro:if value="$(optenv MOVO_HAS_LEFT_ARM_7DOF false)"> <!-- movo has also a left arm of 7 dof type -->
+		    <xacro:jaco_robot_7dof prefix="left_" parent="linear_actuator_link">
+			<origin xyz="0.0261046 0.13335 0.2799937" rpy="${-M_PI/2} 0 ${-M_PI/2}"/>
+		    </xacro:jaco_robot_7dof>
+            	</xacro:if>
+	</xacro:if>
+        <xacro:unless value="$(optenv MOVO_HAS_RIGHT_ARM_7DOF false)" >  <!-- movo has no right arm-->
+		<xacro:if value="$(optenv MOVO_HAS_LEFT_ARM_7DOF false)"> <!-- but has a left arm of 7 dof type -->
+			<xacro:include filename="$(find movo_description)/urdf/manipulation/jaco/jaco_7dof.urdf.xacro" />
+		    	<xacro:jaco_robot_7dof prefix="left_" parent="linear_actuator_link">
+			   <origin xyz="0.0261046 0.13335 0.2799937" rpy="${-M_PI/2} 0 ${-M_PI/2}"/>
+		    	</xacro:jaco_robot_7dof>
+		</xacro:if>
+	</xacro:unless>
+	<xacro:if value="$(optenv MOVO_HAS_RIGHT_ARM_6DOF false)">  <!-- movo has a right arm of 6 dof type -->
+		<xacro:include filename="$(find movo_description)/urdf/manipulation/jaco/jaco.urdf.xacro" />
+		<xacro:jaco_robot prefix="right_" parent="linear_actuator_link">
+		   <origin xyz="0.0261046 -0.13335 0.2799937" rpy="${-M_PI/2} 0 ${-M_PI/2}"/>
+		</xacro:jaco_robot>
+		<xacro:if value="$(optenv MOVO_HAS_LEFT_ARM_6DOF false)"> <!-- movo has also a left arm of 6 dof type -->
+		    <xacro:jaco_robot prefix="left_" parent="linear_actuator_link">
+			<origin xyz="0.0261046 0.13335 0.2799937" rpy="${-M_PI/2} 0 ${-M_PI/2}"/>
 		    </xacro:jaco_robot>
-		    <xacro:if value="$(optenv MOVO_HAS_TWO_KINOVA_ARMS false)">
-		        <xacro:jaco_robot prefix="left_" parent="linear_actuator_link">
-		            <origin xyz="0.0261046 0.13335 0.2799937" rpy="${-M_PI/2} 0 ${-M_PI/2}"/>
-		        </xacro:jaco_robot>
-		    </xacro:if>
-        </xacro:if>
+            	</xacro:if>
+	</xacro:if>
+        <xacro:unless value="$(optenv MOVO_HAS_RIGHT_ARM_6DOF false)" >   <!-- movo has no right arm-->
+		<xacro:if value="$(optenv MOVO_HAS_LEFT_ARM_6DOF false)"> <!-- but has a left arm of 6 dof type -->
+			<xacro:include filename="$(find movo_description)/urdf/manipulation/jaco/jaco.urdf.xacro" />
+		    	<xacro:jaco_robot prefix="left_" parent="linear_actuator_link">
+			   <origin xyz="0.0261046 0.13335 0.2799937" rpy="${-M_PI/2} 0 ${-M_PI/2}"/>
+		    	</xacro:jaco_robot>
+		</xacro:if>
+	</xacro:unless>
         <xacro:if value="$(optenv MOVO_HAS_RIGHT_ROBOTIQ_GRIPPER false)">
             <xacro:robotiq_85_gripper prefix="right_" parent="right_ee_link" >
@@ -120,5 +137,4 @@
             </xacro:kg3_gripper>
         </xacro:if>
-    </xacro:if>
     <xacro:gzplugin_grasp_fix/>
 </robot>
