Commit message: **Work in progress** Modified urdf, created movo_7dof_moveit_config, started work on Gazebo

File: movo_common/movo_description/urdf/movo.urdf.xacro (robot description, xacro)
@@ -32,5 +32,8 @@
     <xacro:include filename="$(find movo_description)/urdf/movo_components/movo_pan_tilt.urdf.xacro" />
     <xacro:include filename="$(find movo_description)/urdf/movo_components/movo_body.urdf.xacro" />
+    <!--
     <xacro:include filename="$(find movo_description)/urdf/manipulation/jaco/jaco.urdf.xacro" />
+    <xacro:include filename="$(find movo_description)/urdf/manipulation/jaco/jaco_7dof.urdf.xacro" />
+    -->
     <xacro:include filename="$(find movo_description)/urdf/manipulation/robotiq/robotiq_85_gripper.urdf.xacro" />
     <xacro:include filename="$(find movo_description)/urdf/manipulation/kinova_grippers/kg3_gripper.urdf.xacro" />
@@ -71,11 +74,23 @@
     <!-- Arms -->
     <xacro:if value="$(optenv MOVO_HAS_KINOVA_ARM false)">
-        <xacro:jaco_robot prefix="right_" parent="linear_actuator_link">
-            <origin xyz="0.0261046 -0.13335 0.2799937" rpy="${-M_PI/2} 0 ${-M_PI/2}"/>
-        </xacro:jaco_robot>
-        <xacro:if value="$(optenv MOVO_HAS_TWO_KINOVA_ARMS false)">
-            <xacro:jaco_robot prefix="left_" parent="linear_actuator_link">
+    	<xacro:if value="$(optenv MOVO_HAS_KINOVA_ARM_7DOF false)">
+    		<xacro:include filename="$(find movo_description)/urdf/manipulation/jaco/jaco_7dof.urdf.xacro" />
+            <xacro:jaco_robot_7dof prefix="left_" parent="linear_actuator_link">
+                <origin xyz="0.0261046 -0.13335 0.2799937" rpy="${-M_PI/2} 0 ${-M_PI/2}"/>
+            </xacro:jaco_robot_7dof>
+            <xacro:jaco_robot_7dof prefix="right_" parent="linear_actuator_link">
                 <origin xyz="0.0261046 0.13335 0.2799937" rpy="${-M_PI/2} 0 ${-M_PI/2}"/>
-            </xacro:jaco_robot>
+            </xacro:jaco_robot_7dof>
+        </xacro:if>
+        <xacro:if value="$(optenv MOVO_HAS_KINOVA_ARM_6DOF false)">
+        	<xacro:include filename="$(find movo_description)/urdf/manipulation/jaco/jaco.urdf.xacro" />
+            <xacro:jaco_robot prefix="right_" parent="linear_actuator_link">
+		        <origin xyz="0.0261046 -0.13335 0.2799937" rpy="${-M_PI/2} 0 ${-M_PI/2}"/>
+		    </xacro:jaco_robot>
+		    <xacro:if value="$(optenv MOVO_HAS_TWO_KINOVA_ARMS false)">
+		        <xacro:jaco_robot prefix="left_" parent="linear_actuator_link">
+		            <origin xyz="0.0261046 0.13335 0.2799937" rpy="${-M_PI/2} 0 ${-M_PI/2}"/>
+		        </xacro:jaco_robot>
+		    </xacro:if>
         </xacro:if>
         <xacro:if value="$(optenv MOVO_HAS_RIGHT_ROBOTIQ_GRIPPER false)">

Commit message: Added IF's in the xacro files to support both cameras

File: movo_common/movo_description/urdf/movo.urdf.xacro (robot description, xacro)
@@ -62,4 +62,5 @@
     </gazebo>
     <xacro:movo_base/>
+    <!-- CHANGE_THIS -->
     <xacro:movo_pan_tilt rgbd_prefix="kinect2" parent="linear_actuator_link">
         <origin xyz="0.19735 0 0.3449888" rpy="0 0 0"/>

File: movo_common/movo_description/urdf/movo_components/movo_pan_tilt.urdf.xacro (robot description, xacro)
@@ -28,5 +28,11 @@
 -->
 <robot name="movo_pan_tilt" xmlns:xacro="http://ros.org/wiki/xacro">
-    <xacro:include filename="$(find movo_description)/urdf/sensors/kinect_one_sensor.urdf.xacro"/>
+	<xacro:if value="$(optenv MOVO_HAS_KINECT_CAMERA false)">
+    	<xacro:include filename="$(find movo_description)/urdf/sensors/kinect_one_sensor.urdf.xacro"/>
+	</xacro:if>
+	<!-- CHANGE_THIS   Add Realsense description -->
+	<xacro:if value="$(optenv MOVO_HAS_REALSENSE_CAMERA false)">
+    	<!--xacro:include filename="$(find movo_description)/urdf/sensors/kinect_one_sensor.urdf.xacro"/-->
+	</xacro:if>
     <xacro:property name="M_PI" value="3.14159"/>
     <xacro:macro name="movo_pan_tilt" params="rgbd_prefix parent *origin">
@@ -126,7 +132,17 @@
             </inertial>
 		</link>
-		<xacro:kinect_one_sensor prefix="${rgbd_prefix}" parent="tilt_link">
-			<origin xyz="0.05825 -0.0105875 -0.026" rpy="${-M_PI/2} 0 ${-M_PI/2}" />
-		</xacro:kinect_one_sensor>
+       	<xacro:if value="$(optenv MOVO_HAS_KINECT_CAMERA false)">
+			<xacro:kinect_one_sensor prefix="${rgbd_prefix}" parent="tilt_link">
+				<origin xyz="0.05825 -0.0105875 -0.026" rpy="${-M_PI/2} 0 ${-M_PI/2}" />
+			</xacro:kinect_one_sensor>
+		</xacro:if>
+		<!-- CHANGE_THIS call the realsense object -->
+		<xacro:if value="$(optenv MOVO_HAS_REALSENSE_CAMERA false)">
+			<!--
+			<xacro:kinect_one_sensor prefix="${rgbd_prefix}" parent="tilt_link">
+				<origin xyz="0.05825 -0.0105875 -0.026" rpy="${-M_PI/2} 0 ${-M_PI/2}" />
+			</xacro:kinect_one_sensor>
+			-->
+		</xacro:if>
     </xacro:macro>
 </robot>

File: movo_common/movo_description/urdf/pan_tilt_stand_alone.urdf.xacro (robot description, xacro)
@@ -36,6 +36,11 @@
     </gazebo>
     <link name="root"/>
-    <xacro:movo_pan_tilt rgbd_prefix="kinect" parent="root">
-        <origin xyz="0.19735 0 0.3449888" rpy="0 0 0"/>
-    </xacro:movo_pan_tilt>
+    <!-- CHANGE_THIS -->
+    <xacro:if value="$(optenv MOVO_HAS_KINECT_CAMERA false)">
+      <xacro:movo_pan_tilt rgbd_prefix="kinect" parent="root">
+          <origin xyz="0.19735 0 0.3449888" rpy="0 0 0"/>
+      </xacro:movo_pan_tilt>
+    </xacro:if>
+    <xacro:if value="$(optenv MOVO_HAS_REALSENSE_CAMERA false)">
+ 		</xacro:if>
 </robot>

File: movo_common/movo_description/urdf/sensors/kinect_one_sensor.urdf.xacro (robot description, xacro)
@@ -28,4 +28,5 @@
 -->
 <robot xmlns:xacro="http://ros.org/wiki/xacro" name="kinect_one_sensor">
+    <!-- CHANGE_THIS -->
 	<xacro:macro name="kinect_one_sensor" params="prefix parent *origin">
         <joint name="${prefix}_joint" type="fixed">

Commit message: Change link names and change topic remapping so if either camera is used, the same generic topic names are used

File: movo_common/movo_description/urdf/movo.urdf.xacro (robot description, xacro)
@@ -62,5 +62,4 @@
     </gazebo>
     <xacro:movo_base/>
-    <!-- CHANGE_THIS -->
     <xacro:movo_pan_tilt rgbd_prefix="camera" parent="linear_actuator_link">
         <origin xyz="0.19735 0 0.3449888" rpy="0 0 0"/>

File: movo_common/movo_description/urdf/movo_components/movo_pan_tilt.urdf.xacro (robot description, xacro)
@@ -28,10 +28,12 @@
 -->
 <robot name="movo_pan_tilt" xmlns:xacro="http://ros.org/wiki/xacro">
+	<!-- MOVO Camera -->
+	<!-- Kinect is the camera -->
 	<xacro:if value="$(optenv MOVO_HAS_KINECT_CAMERA false)">
     	<xacro:include filename="$(find movo_description)/urdf/sensors/kinect_one_sensor.urdf.xacro"/>
 	</xacro:if>
-	<!-- CHANGE_THIS   Add Realsense description -->
+	<!-- Realsense is the camera -->
 	<xacro:if value="$(optenv MOVO_HAS_REALSENSE_CAMERA false)">
-    	<!--xacro:include filename="$(find movo_description)/urdf/sensors/kinect_one_sensor.urdf.xacro"/-->
+    	<xacro:include filename="$(find movo_description)/urdf/sensors/_r430.urdf.xacro"/>
 	</xacro:if>
     <xacro:property name="M_PI" value="3.14159"/>
@@ -132,16 +134,15 @@
             </inertial>
 		</link>
-       	<xacro:if value="$(optenv MOVO_HAS_KINECT_CAMERA false)">
+       	<!-- Camera is Kinect One -->
+		<xacro:if value="$(optenv MOVO_HAS_KINECT_CAMERA false)">
 			<xacro:kinect_one_sensor prefix="${rgbd_prefix}" parent="tilt_link">
 				<origin xyz="0.05825 -0.0105875 -0.026" rpy="${-M_PI/2} 0 ${-M_PI/2}" />
 			</xacro:kinect_one_sensor>
 		</xacro:if>
-		<!-- CHANGE_THIS call the realsense object -->
+		<!-- Camera is Realsense -->
 		<xacro:if value="$(optenv MOVO_HAS_REALSENSE_CAMERA false)">
-			<!--
-			<xacro:kinect_one_sensor prefix="${rgbd_prefix}" parent="tilt_link">
+			<xacro:sensor_r430 prefix="${rgbd_prefix}" parent="tilt_link">
 				<origin xyz="0.05825 -0.0105875 -0.026" rpy="${-M_PI/2} 0 ${-M_PI/2}" />
-			</xacro:kinect_one_sensor>
-			-->
+			</xacro:sensor_r430>
 		</xacro:if>
     </xacro:macro>

File: movo_common/movo_description/urdf/pan_tilt_stand_alone.urdf.xacro (robot description, xacro)
@@ -36,11 +36,6 @@
     </gazebo>
     <link name="root"/>
-    <!-- CHANGE_THIS -->
-    <xacro:if value="$(optenv MOVO_HAS_KINECT_CAMERA false)">
-      <xacro:movo_pan_tilt rgbd_prefix="camera" parent="root">
-          <origin xyz="0.19735 0 0.3449888" rpy="0 0 0"/>
-      </xacro:movo_pan_tilt>
-    </xacro:if>
-    <xacro:if value="$(optenv MOVO_HAS_REALSENSE_CAMERA false)">
- 		</xacro:if>
+    <xacro:movo_pan_tilt rgbd_prefix="camera" parent="root">
+        <origin xyz="0.19735 0 0.3449888" rpy="0 0 0"/>
+    </xacro:movo_pan_tilt>
 </robot>

File: movo_common/movo_description/urdf/sensors/kinect_one_sensor.urdf.xacro (robot description, xacro)
@@ -54,8 +54,8 @@
 			</collision>
 		</link>
-        <link name="${prefix}_ir_link"/>
+        <link name="${prefix}_ir_frame"/>
         <joint name="${prefix}_ir_joint" type="fixed">
             <parent link="${prefix}_link"/>
-            <child link="${prefix}_ir_link" />
+            <child link="${prefix}_ir_frame" />
             <origin xyz="0.0245 -0.03325  0.04201" rpy="0 0 0"/>
         </joint>
@@ -63,16 +63,16 @@
         <joint name="${prefix}_ir_optical_frame_joint" type="fixed">
             <origin xyz="0 0 0" rpy="${-M_PI / 2.0} 0 ${-M_PI / 2.0}" />
-            <parent link="${prefix}_ir_link"/>
+            <parent link="${prefix}_ir_frame"/>
             <child link="${prefix}_ir_optical_frame"/>
         </joint>
-        <link name="${prefix}_color_link"/>
+        <link name="${prefix}_color_frame"/>
         <joint name="${prefix}_color_joint" type="fixed">
-            <parent link="${prefix}_ir_link"/>
-            <child link="${prefix}_color_link" />
+            <parent link="${prefix}_ir_frame"/>
+            <child link="${prefix}_color_frame" />
             <origin xyz="0 -0.06175  0" rpy="0 0 0"/>
         </joint>
         <link name="${prefix}_color_optical_frame"/>
         <joint name="${prefix}_color_optical_joint" type="fixed">
-            <parent link="${prefix}_color_link"/>
+            <parent link="${prefix}_color_frame"/>
             <child link="${prefix}_color_optical_frame" />
             <origin xyz="0 0 0" rpy="${-M_PI / 2.0} 0 ${-M_PI / 2.0}"/>

File: movo_common/movo_third_party/realsense2_camera/urdf/_r410.urdf.xacro (robot description, xacro)
@@ -27,12 +27,12 @@
     <color rgba="0.5 0.5 0.5 1"/>
   </material>
-  <xacro:macro name="sensor_r410" params="parent *origin">
+  <xacro:macro name="sensor_r410" params="prefix parent *origin">
     <!-- camera body, with origin at bottom screw mount -->
-    <joint name="camera_joint" type="fixed">
+    <joint name="${prefix}_joint" type="fixed">
       <xacro:insert_block name="origin" />
       <parent link="${parent}"/>
-      <child link="camera_link" />
+      <child link="${prefix}_link" />
     </joint>
-    <link name="camera_link">
+    <link name="${prefix}_link">
       <visual>
       <origin xyz="0 ${-r410_cam_mount_from_center_offset} ${r410_cam_height/2}" rpy="${M_PI/2} 0 ${M_PI/2}"/>
@@ -57,42 +57,42 @@
     </link>
     <!-- camera depth joints and links -->
-    <joint name="camera_depth_joint" type="fixed">
+    <joint name="${prefix}_depth_joint" type="fixed">
       <origin xyz="${r410_cam_depth_px} ${r410_cam_depth_py} ${r410_cam_depth_pz}" rpy="0 0 0"/>
-      <parent link="camera_link"/>
-      <child link="camera_depth_frame" />
+      <parent link="${prefix}_link"/>
+      <child link="${prefix}_depth_frame" />
     </joint>
-    <link name="camera_depth_frame"/>
-    <joint name="camera_depth_optical_joint" type="fixed">
+    <link name="${prefix}_depth_frame"/>
+    <joint name="${prefix}_depth_optical_joint" type="fixed">
       <origin xyz="0 0 0" rpy="${-M_PI/2} 0 ${-M_PI/2}" />
-      <parent link="camera_depth_frame" />
-      <child link="camera_depth_optical_frame" />
+      <parent link="${prefix}_depth_frame" />
+      <child link="${prefix}_depth_optical_frame" />
     </joint>
-    <link name="camera_depth_optical_frame"/>
+    <link name="${prefix}_depth_optical_frame"/>
     <!-- camera left IR joints and links -->
-    <joint name="camera_left_ir_joint" type="fixed">
+    <joint name="${prefix}_left_ir_joint" type="fixed">
       <origin xyz="0 ${r410_cam_depth_to_left_ir_offset} 0" rpy="0 0 0" />
-      <parent link="camera_depth_frame" />
-      <child link="camera_left_ir_frame" />
+      <parent link="${prefix}_depth_frame" />
+      <child link="${prefix}_left_ir_frame" />
     </joint>
-    <link name="camera_left_ir_frame"/>
-    <joint name="camera_left_ir_optical_joint" type="fixed">
+    <link name="${prefix}_left_ir_frame"/>
+    <joint name="${prefix}_left_ir_optical_joint" type="fixed">
       <origin xyz="0 0 0" rpy="${-M_PI/2} 0 ${-M_PI/2}" />
-      <parent link="camera_left_ir_frame" />
-      <child link="camera_left_ir_optical_frame" />
+      <parent link="${prefix}_left_ir_frame" />
+      <child link="${prefix}_left_ir_optical_frame" />
     </joint>
-    <link name="camera_left_ir_optical_frame"/>
+    <link name="${prefix}_left_ir_optical_frame"/>
     <!-- camera right IR joints and links -->
-    <joint name="camera_right_ir_joint" type="fixed">
+    <joint name="${prefix}_right_ir_joint" type="fixed">
       <origin xyz="0 ${r410_cam_depth_to_right_ir_offset} 0" rpy="0 0 0" />
-      <parent link="camera_depth_frame" />
-      <child link="camera_right_ir_frame" />
+      <parent link="${prefix}_depth_frame" />
+      <child link="${prefix}_right_ir_frame" />
     </joint>
-    <link name="camera_right_ir_frame"/>
-    <joint name="camera_right_ir_optical_joint" type="fixed">
+    <link name="${prefix}_right_ir_frame"/>
+    <joint name="${prefix}_right_ir_optical_joint" type="fixed">
       <origin xyz="0 0 0" rpy="${-M_PI/2} 0 ${-M_PI/2}" />
-      <parent link="camera_right_ir_frame" />
-      <child link="camera_right_ir_optical_frame" />
+      <parent link="${prefix}_right_ir_frame" />
+      <child link="${prefix}_right_ir_optical_frame" />
     </joint>
-    <link name="camera_right_ir_optical_frame"/>
+    <link name="${prefix}_right_ir_optical_frame"/>
   </xacro:macro>
 </robot>

File: movo_common/movo_third_party/realsense2_camera/urdf/test_r410_camera.urdf.xacro (robot description, xacro)
@@ -3,5 +3,5 @@
   <xacro:include filename="$(find realsense2_camera)/urdf/_r410.urdf.xacro"/>
   <link name="base_link" />
-  <sensor_r410 parent="base_link">
+  <sensor_r410 prefix="camera_" parent="base_link">
     <origin xyz="0 0 0" rpy="0 0 0"/>
   </sensor_r410>

File: movo_common/movo_third_party/realsense2_camera/urdf/test_r430_camera.urdf.xacro (robot description, xacro)
@@ -3,5 +3,5 @@
   <xacro:include filename="$(find realsense2_camera)/urdf/_r430.urdf.xacro"/>
   <link name="base_link" />
-  <sensor_r430 parent="base_link">
+  <sensor_r430 prefix="camera_" parent="base_link">
     <origin xyz="0 0 0" rpy="0 0 0"/>
   </sensor_r430>

Commit message: modified files first implementation untested

File: movo_common/movo_description/urdf/movo.urdf.xacro (robot description, xacro)
@@ -69,25 +69,42 @@
     </xacro:if>
     <!-- Arms -->
-    <xacro:if value="$(optenv MOVO_HAS_KINOVA_ARM false)">
-    	<xacro:if value="$(optenv MOVO_HAS_KINOVA_ARM_7DOF false)">
-    		<xacro:include filename="$(find movo_description)/urdf/manipulation/jaco/jaco_7dof.urdf.xacro" />
-            <xacro:jaco_robot_7dof prefix="right_" parent="linear_actuator_link">
-            <origin xyz="0.0261046 -0.13335 0.2799937" rpy="${-M_PI/2} 0 ${-M_PI/2}"/>
-            </xacro:jaco_robot_7dof>
-            <xacro:jaco_robot_7dof prefix="left_" parent="linear_actuator_link">
-                <origin xyz="0.0261046 0.13335 0.2799937" rpy="${-M_PI/2} 0 ${-M_PI/2}"/>
-            </xacro:jaco_robot_7dof>
-        </xacro:if>
-        <xacro:if value="$(optenv MOVO_HAS_KINOVA_ARM_6DOF false)">
-        	<xacro:include filename="$(find movo_description)/urdf/manipulation/jaco/jaco.urdf.xacro" />
-            <xacro:jaco_robot prefix="right_" parent="linear_actuator_link">
-		        <origin xyz="0.0261046 -0.13335 0.2799937" rpy="${-M_PI/2} 0 ${-M_PI/2}"/>
+	<xacro:if value="$(optenv MOVO_HAS_RIGHT_ARM_7DOF false)">  <!-- movo has a right arm of 7 dof type -->
+		<xacro:include filename="$(find movo_description)/urdf/manipulation/jaco/jaco_7dof.urdf.xacro" />
+		<xacro:jaco_robot_7dof prefix="right_" parent="linear_actuator_link">
+		   <origin xyz="0.0261046 -0.13335 0.2799937" rpy="${-M_PI/2} 0 ${-M_PI/2}"/>
+		</xacro:jaco_robot_7dof>
+		<xacro:if value="$(optenv MOVO_HAS_LEFT_ARM_7DOF false)"> <!-- movo has also a left arm of 7 dof type -->
+		    <xacro:jaco_robot_7dof prefix="left_" parent="linear_actuator_link">
+			<origin xyz="0.0261046 0.13335 0.2799937" rpy="${-M_PI/2} 0 ${-M_PI/2}"/>
+		    </xacro:jaco_robot_7dof>
+            	</xacro:if>
+	</xacro:if>
+        <xacro:unless value="$(optenv MOVO_HAS_RIGHT_ARM_7DOF false)" >  <!-- movo has no right arm-->
+		<xacro:if value="$(optenv MOVO_HAS_LEFT_ARM_7DOF false)"> <!-- but has a left arm of 7 dof type -->
+			<xacro:include filename="$(find movo_description)/urdf/manipulation/jaco/jaco_7dof.urdf.xacro" />
+		    	<xacro:jaco_robot_7dof prefix="left_" parent="linear_actuator_link">
+			   <origin xyz="0.0261046 0.13335 0.2799937" rpy="${-M_PI/2} 0 ${-M_PI/2}"/>
+		    	</xacro:jaco_robot_7dof>
+		</xacro:if>
+	</xacro:unless>
+	<xacro:if value="$(optenv MOVO_HAS_RIGHT_ARM_6DOF false)">  <!-- movo has a right arm of 6 dof type -->
+		<xacro:include filename="$(find movo_description)/urdf/manipulation/jaco/jaco.urdf.xacro" />
+		<xacro:jaco_robot prefix="right_" parent="linear_actuator_link">
+		   <origin xyz="0.0261046 -0.13335 0.2799937" rpy="${-M_PI/2} 0 ${-M_PI/2}"/>
+		</xacro:jaco_robot>
+		<xacro:if value="$(optenv MOVO_HAS_LEFT_ARM_6DOF false)"> <!-- movo has also a left arm of 6 dof type -->
+		    <xacro:jaco_robot prefix="left_" parent="linear_actuator_link">
+			<origin xyz="0.0261046 0.13335 0.2799937" rpy="${-M_PI/2} 0 ${-M_PI/2}"/>
 		    </xacro:jaco_robot>
-		    <xacro:if value="$(optenv MOVO_HAS_TWO_KINOVA_ARMS false)">
-		        <xacro:jaco_robot prefix="left_" parent="linear_actuator_link">
-		            <origin xyz="0.0261046 0.13335 0.2799937" rpy="${-M_PI/2} 0 ${-M_PI/2}"/>
-		        </xacro:jaco_robot>
-		    </xacro:if>
-        </xacro:if>
+            	</xacro:if>
+	</xacro:if>
+        <xacro:unless value="$(optenv MOVO_HAS_RIGHT_ARM_6DOF false)" >   <!-- movo has no right arm-->
+		<xacro:if value="$(optenv MOVO_HAS_LEFT_ARM_6DOF false)"> <!-- but has a left arm of 6 dof type -->
+			<xacro:include filename="$(find movo_description)/urdf/manipulation/jaco/jaco.urdf.xacro" />
+		    	<xacro:jaco_robot prefix="left_" parent="linear_actuator_link">
+			   <origin xyz="0.0261046 0.13335 0.2799937" rpy="${-M_PI/2} 0 ${-M_PI/2}"/>
+		    	</xacro:jaco_robot>
+		</xacro:if>
+	</xacro:unless>
         <xacro:if value="$(optenv MOVO_HAS_RIGHT_ROBOTIQ_GRIPPER false)">
             <xacro:robotiq_85_gripper prefix="right_" parent="right_ee_link" >
@@ -120,5 +137,4 @@
             </xacro:kg3_gripper>
         </xacro:if>
-    </xacro:if>
     <xacro:gzplugin_grasp_fix/>
 </robot>
