Commit message: Added some parameters to the Realsense node launch file to match frames and links. Still got to fix the robot model and remap topics to the right names for the Realsense

File: movo_common/movo_description/urdf/movo_components/movo_pan_tilt.urdf.xacro (robot description, xacro)
@@ -35,4 +35,5 @@
 	<!-- Realsense is the camera -->
 	<xacro:if value="$(optenv MOVO_HAS_REALSENSE_CAMERA false)">
+		<xacro:include filename="$(find movo_description)/urdf/sensors/_r410.urdf.xacro"/>
     	<xacro:include filename="$(find movo_description)/urdf/sensors/_r430.urdf.xacro"/>
 	</xacro:if>
@@ -142,7 +143,7 @@
 		<!-- Camera is Realsense -->
 		<xacro:if value="$(optenv MOVO_HAS_REALSENSE_CAMERA false)">
-			<xacro:sensor_r430 prefix="${rgbd_prefix}" parent="tilt_link">
+			<xacro:sensor_r410 prefix="${rgbd_prefix}" parent="tilt_link">
 				<origin xyz="0.05825 -0.0105875 -0.026" rpy="${-M_PI/2} 0 ${-M_PI/2}" />
-			</xacro:sensor_r430>
+			</xacro:sensor_r410>
 		</xacro:if>
     </xacro:macro>

File: movo_common/movo_description/urdf/pan_tilt_stand_alone.urdf.xacro (robot description, xacro)
@@ -36,5 +36,5 @@
     </gazebo>
     <link name="root"/>
-    <xacro:movo_pan_tilt rgbd_prefix="camera" parent="root">
+    <xacro:movo_pan_tilt rgbd_prefix="movo_camera" parent="root">
         <origin xyz="0.19735 0 0.3449888" rpy="0 0 0"/>
     </xacro:movo_pan_tilt>

File: movo_common/movo_description/urdf/sensors/_r410.urdf.xacro (robot description, xacro)
@@ -3,30 +3,29 @@
 License: Apache 2.0. See LICENSE file in root directory.
 Copyright(c) 2017 Intel Corporation. All Rights Reserved
-This is the URDF model for the Intel RealSense 430 camera, in it's
-aluminum peripherial evaluation case.
+This is the URDF model for the Intel RealSense 410 camera, in it's
+aluminum peripherial evalution case.
 -->
-<robot name="sensor_r430" xmlns:xacro="http://ros.org/wiki/xacro">
+<robot name="sensor_r410" xmlns:xacro="http://ros.org/wiki/xacro">
   <xacro:property name="M_PI" value="3.1415926535897931" />
   <!-- The following values are approximate, and the camera node
    publishing TF values with actual calibrated camera extrinsic values -->
-  <xacro:property name="r430_cam_depth_to_left_ir_offset" value="-0.025"/>
-  <xacro:property name="r430_cam_depth_to_right_ir_offset" value="0.025"/>
-  <xacro:property name="r430_cam_depth_to_fisheye_offset" value="0.042"/>
+  <xacro:property name="r410_cam_depth_to_left_ir_offset" value="-0.0275"/>
+  <xacro:property name="r410_cam_depth_to_right_ir_offset" value="0.0275"/>
   <!-- The following values model the aluminum peripherial case for the
-    R430 camera, with the camera joint represented by the actual
+    R410 camera, with the camera joint represented by the actual
     peripherial camera tripod mount -->
-  <xacro:property name="r430_cam_width" value="0.105"/>
-  <xacro:property name="r430_cam_height" value="0.039"/>
-  <xacro:property name="r430_cam_depth" value="0.019"/>
-  <xacro:property name="r430_cam_mount_from_center_offset" value=".0275"/>
-  <!-- The following offset is relative the the physical R430 camera peripherial
+  <xacro:property name="r410_cam_width" value="0.099"/>
+  <xacro:property name="r410_cam_height" value="0.035"/>
+  <xacro:property name="r410_cam_depth" value="0.0185"/>
+  <xacro:property name="r410_cam_mount_from_center_offset" value=".0375"/>
+  <!-- The following offset is relative the the physical R410 camera peripherial
     camera tripod mount -->
-  <xacro:property name="r430_cam_depth_px" value="0.00"/>
-  <xacro:property name="r430_cam_depth_py" value="-0.035"/>
-  <xacro:property name="r430_cam_depth_pz" value="0.028"/>
+  <xacro:property name="r410_cam_depth_px" value="0.00"/>
+  <xacro:property name="r410_cam_depth_py" value="-0.0425"/>
+  <xacro:property name="r410_cam_depth_pz" value="0.026"/>
   <!-- <material name="aluminum">
     <color rgba="0.5 0.5 0.5 1"/>
   </material> -->
-  <xacro:macro name="sensor_r430" params="prefix parent *origin">
+  <xacro:macro name="sensor_r410" params="prefix parent *origin">
     <!-- camera body, with origin at bottom screw mount -->
     <joint name="${prefix}_joint" type="fixed">
@@ -37,15 +36,15 @@
     <link name="${prefix}_link">
       <visual>
-      <origin xyz="0 ${-r430_cam_mount_from_center_offset} ${r430_cam_height/2}" rpy="${M_PI/2} 0 ${M_PI/2}"/>
+      <origin xyz="0 ${-r410_cam_mount_from_center_offset} ${r410_cam_height/2}" rpy="${M_PI/2} 0 ${M_PI/2}"/>
         <geometry>
-          <box size="${r430_cam_width} ${r430_cam_height} ${r430_cam_depth}"/>
-          <!--<mesh filename="package://realsense2_camera/meshes/r430/r430.dae" />-->
+          <box size="${r410_cam_width} ${r410_cam_height} ${r410_cam_depth}"/>
+          <!--<mesh filename="package://realsense2_camera/meshes/r410/r410.dae" />-->
         </geometry>
         <!-- <material name="aluminum"/> -->
       </visual>
       <collision>
-        <origin xyz="0.0 0.0 ${r430_cam_height/2}" rpy="0 0 0"/>
+        <origin xyz="0.0 0.0 ${r410_cam_height/2}" rpy="0 0 0"/>
         <geometry>
-        <box size="${r430_cam_depth} ${r430_cam_width} ${r430_cam_height}"/>
+        <box size="${r410_cam_depth} ${r410_cam_width} ${r410_cam_height}"/>
         </geometry>
       </collision>
@@ -59,5 +58,5 @@
     <!-- camera depth joints and links -->
     <joint name="${prefix}_depth_joint" type="fixed">
-      <origin xyz="${r430_cam_depth_px} ${r430_cam_depth_py} ${r430_cam_depth_pz}" rpy="0 0 0"/>
+      <origin xyz="${r410_cam_depth_px} ${r410_cam_depth_py} ${r410_cam_depth_pz}" rpy="0 0 0"/>
       <parent link="${prefix}_link"/>
       <child link="${prefix}_depth_frame" />
@@ -72,5 +71,5 @@
     <!-- camera left IR joints and links -->
     <joint name="${prefix}_left_ir_joint" type="fixed">
-      <origin xyz="0 ${r430_cam_depth_to_left_ir_offset} 0" rpy="0 0 0" />
+      <origin xyz="0 ${r410_cam_depth_to_left_ir_offset} 0" rpy="0 0 0" />
       <parent link="${prefix}_depth_frame" />
       <child link="${prefix}_left_ir_frame" />
@@ -85,5 +84,5 @@
     <!-- camera right IR joints and links -->
     <joint name="${prefix}_right_ir_joint" type="fixed">
-      <origin xyz="0 ${r430_cam_depth_to_right_ir_offset} 0" rpy="0 0 0" />
+      <origin xyz="0 ${r410_cam_depth_to_right_ir_offset} 0" rpy="0 0 0" />
       <parent link="${prefix}_depth_frame" />
       <child link="${prefix}_right_ir_frame" />
@@ -96,17 +95,4 @@
     </joint>
     <link name="${prefix}_right_ir_optical_frame"/>
-    <!-- camera fisheye joints and links -->
-    <joint name="${prefix}_fisheye_joint" type="fixed">
-      <origin xyz="0 ${r430_cam_depth_to_fisheye_offset} 0" rpy="0 0 0" />
-      <parent link="${prefix}_depth_frame" />
-      <child link="${prefix}_fisheye_frame" />
-    </joint>
-    <link name="${prefix}_fisheye_frame"/>
-    <joint name="${prefix}_fisheye_optical_joint" type="fixed">
-      <origin xyz="0 0 0" rpy="${-M_PI/2} 0 ${-M_PI/2}" />
-      <parent link="${prefix}_fisheye_frame" />
-      <child link="${prefix}_fisheye_optical_frame" />
-    </joint>
-    <link name="${prefix}_fisheye_optical_frame"/>
   </xacro:macro>
 </robot>

Commit message: Now the robot model is not realistic but almost when using realsense as the camera

File: movo_common/movo_description/urdf/movo_components/movo_pan_tilt.urdf.xacro (robot description, xacro)
@@ -144,5 +144,5 @@
 		<xacro:if value="$(optenv MOVO_HAS_REALSENSE_CAMERA false)">
 			<xacro:sensor_r410 prefix="${rgbd_prefix}" parent="tilt_link">
-				<origin xyz="0.05825 -0.0105875 -0.026" rpy="${-M_PI/2} 0 ${-M_PI/2}" />
+				<origin xyz="0.05825 -0.02 -0.065" rpy="${-M_PI/2} 0 ${-M_PI/2}" />
 			</xacro:sensor_r410>
 		</xacro:if>

File: movo_common/movo_description/urdf/sensors/_r410.urdf.xacro (robot description, xacro)
@@ -24,7 +24,7 @@
   <xacro:property name="r410_cam_depth_py" value="-0.0425"/>
   <xacro:property name="r410_cam_depth_pz" value="0.026"/>
-  <!-- <material name="aluminum">
-    <color rgba="0.5 0.5 0.5 1"/>
-  </material> -->
+  <material name="rs_gray">
+    <color rgba="0.75 0.75 0.75 1"/>
+  </material>
   <xacro:macro name="sensor_r410" params="prefix parent *origin">
     <!-- camera body, with origin at bottom screw mount -->
@@ -41,5 +41,5 @@
           <!--<mesh filename="package://realsense2_camera/meshes/r410/r410.dae" />-->
         </geometry>
-        <!-- <material name="aluminum"/> -->
+        <material name="rs_gray"/>
       </visual>
       <collision>

Commit message: Change from kinect to realsense for perception launch
replace some kinect point topics

Replace kinect2 with d435 for srdf ignore collisions

Remove most kinect files

Add some realsense model files

Change d435_link to camera_link

Change kinect ptclouds to camera/depth/color/points

Replace kinect with d435 in xacro files

Replace run dependecy on iai_kinect with realsense-ros

Remove kinect collision stl

Remap default_pointing_frame to realsense camera_link

Replace kinect rviz file references with realsense

Remove kinect install dependency

Try to add variable to launch pointcloud

Fix urdf.xacro file issues

Adjust realsense position in urdf

Remove kinect collision file

File: movo_common/movo_description/urdf/movo_components/movo_pan_tilt.urdf.xacro (robot description, xacro)
@@ -2,5 +2,5 @@
 <!--
 Software License Agreement (BSD)
-\file      pan_tilt_kinect_one.urdf.xacro
+\file      pan_tilt_d435.urdf.xacro
 \authors   Patrick Hussey
 \copyright Copyright (c) 2017, Kinova Robotics inc. All rights reserved.
@@ -28,5 +28,5 @@
 -->
 <robot name="movo_pan_tilt" xmlns:xacro="http://ros.org/wiki/xacro">
-    <xacro:include filename="$(find movo_description)/urdf/sensors/kinect_one_sensor.urdf.xacro"/>
+    <xacro:include filename="$(find movo_description)/urdf/sensors/_d435.urdf.xacro"/>
     <xacro:property name="M_PI" value="3.14159"/>
     <xacro:macro name="movo_pan_tilt" params="rgbd_prefix parent *origin">
@@ -126,7 +126,7 @@
             </inertial>
 		</link>
-		<xacro:kinect_one_sensor prefix="${rgbd_prefix}" parent="tilt_link">
-			<origin xyz="0.05825 -0.0105875 -0.026" rpy="${-M_PI/2} 0 ${-M_PI/2}" />
-		</xacro:kinect_one_sensor>
+		<xacro:sensor_d435 parent="tilt_link">
+			<origin xyz="0.06 0 -0.025" rpy="${-M_PI/2} 0 ${-M_PI/2}" />
+		</xacro:sensor_d435>
     </xacro:macro>
 </robot>

Commit message: Add point cloud. Adjust camera optical joint positions

File: movo_common/movo_description/urdf/movo_components/movo_pan_tilt.urdf.xacro (robot description, xacro)
@@ -129,5 +129,5 @@
 		</link>
 		<xacro:sensor_d435 parent="tilt_link">
-			<origin xyz="0.06 0 -0.025" rpy="${-M_PI/2} 0 ${-M_PI/2}" />
+			<origin xyz="0.08 0 -0.025" rpy="${-M_PI/2} 0 ${-M_PI/2}" />
 		</xacro:sensor_d435>
     </xacro:macro>

File: movo_common/movo_description/urdf/sensors/_d435.gazebo.xacro (robot description, xacro)
@@ -131,6 +131,6 @@
       	<rangeMinDepth>0.2</rangeMinDepth>
       	<rangeMaxDepth>10.0</rangeMaxDepth>
-      	<pointCloud>false</pointCloud>
-      	<pointCloudTopicName>depth/points</pointCloudTopicName>
+      	<pointCloud>true</pointCloud>
+	<pointCloudTopicName>depth/color/points</pointCloudTopicName>
       	<pointCloudCutoff>0.5</pointCloudCutoff>
       </plugin>

File: movo_common/movo_description/urdf/sensors/_d435_sim.urdf.xacro (robot description, xacro)
@@ -74,5 +74,5 @@
     <link name="${name}_depth_frame"/>
     <joint name="${name}_depth_optical_joint" type="fixed">
-      <origin xyz="0 0 0" rpy="${-M_PI/2} 0 ${-M_PI/2}" />
+      <origin xyz="0.005 0 0" rpy="${-M_PI/2} 0 ${-M_PI/2}" />
       <parent link="${name}_depth_frame" />
       <child link="${name}_depth_optical_frame" />
@@ -87,5 +87,5 @@
     <link name="${name}_left_ir_frame"/>
     <joint name="${name}_left_ir_optical_joint" type="fixed">
-      <origin xyz="0 0 0" rpy="${-M_PI/2} 0 ${-M_PI/2}" />
+      <origin xyz="0.005 0 0" rpy="${-M_PI/2} 0 ${-M_PI/2}" />
       <parent link="${name}_left_ir_frame" />
       <child link="${name}_left_ir_optical_frame" />
@@ -100,5 +100,5 @@
     <link name="${name}_right_ir_frame"/>
     <joint name="${name}_right_ir_optical_joint" type="fixed">
-      <origin xyz="0 0 0" rpy="${-M_PI/2} 0 ${-M_PI/2}" />
+      <origin xyz="0.005 0 0" rpy="${-M_PI/2} 0 ${-M_PI/2}" />
       <parent link="${name}_right_ir_frame" />
       <child link="${name}_right_ir_optical_frame" />
@@ -113,5 +113,5 @@
     <link name="${name}_color_frame"/>
     <joint name="${name}_color_optical_joint" type="fixed">
-      <origin xyz="0 0 0" rpy="${-M_PI/2} 0 ${-M_PI/2}" />
+      <origin xyz="0.005 0 0" rpy="${-M_PI/2} 0 ${-M_PI/2}" />
       <parent link="${name}_color_frame" />
       <child link="${name}_color_optical_frame" />
@@ -120,4 +120,4 @@
     <!-- Realsense Gazebo Plugin -->
     <xacro:gazebo_d435 camera_name="${name}" reference_link="${name}_link" topics_ns="${topics_ns}" depth_optical_frame="${name}_depth_optical_frame" color_optical_frame="${name}_color_optical_frame" infrared1_optical_frame="${name}_left_ir_optical_frame" infrared2_optical_frame="${name}_right_ir_optical_frame"/>
-  </xacro:macro>
+    </xacro:macro>
 </robot>
